Commit message: integrating gripper and adding explanatory comments in the code

File: models/objects/finger_tool.urdf.xacro (robot description, xacro)
@@ -2,4 +2,5 @@
 <robot xmlns:xacro="http://www.ros.org/wiki/xacro" name="finger_tool">
     <xacro:property name="PI" value="3.14159265359" />
+    <xacro:property name="scale_factor" value="0.001" />
     <!-- Base link -->
     <link name="tool_base">
@@ -8,5 +9,5 @@
             <origin xyz="0 0 0" rpy="${PI/2} 0.0 0.0"/>
             <geometry>
-                <mesh filename="package://robot_arm_motion/models/objects/meshes/fingerTool.STL" scale="0.001 0.001 0.001"/>
+                <mesh filename="package://robot_arm_motion/models/objects/meshes/fingerTool.STL" scale="${scale_factor} ${scale_factor} ${scale_factor}"/>
             </geometry>
             <material name="black">
@@ -15,9 +16,3 @@
         </visual>
     </link>
-    <!-- <joint name="joint_tool" type="revolute">
-        <axis xyz="0 0 1"/>
-        <limit effort="15" lower="-0.47" upper="0.47" velocity="7"/>
-        <parent link="tool_base"/>
-        <origin xyz="0 0 0" rpy="0 0 0"/>
-    </joint> -->
 </robot>
